File: EnvelopeFollower.sch (KiCad schematic (older format))
At the start: 84 parts, among them J1 RTip, J10 IN, J11 GND, J12 GND, J13 SW1B, J14 OUT, J15 DTIP, J16 DSW, J17 GND, J18 ITIP, J19 ISLV, J20 SW1C, J3 +9v, J4 GND, J5 SEND, J6 RSLV, J7 GND, J8 GND, J9 SW1A, SW1 Moog, SW2 BANDWIDTH, SW3 MODE, U1 TL074, U2 LM1458, U3 VTL5C, U4 VTL5C

Commit message: V2.00 provisionaly completed
Parts:
- removed J13: SW1B, Connector_Wire:SolderWire-0.25sqmm_1x03_P4.2mm_D0.65mm_OD1.7mm, symbol Connector_Generic:Conn_01x03
- removed J20: SW1C, Connector_Wire:SolderWire-0.25sqmm_1x03_P4.2mm_D0.65mm_OD1.7mm, symbol Connector_Generic:Conn_01x03
- removed J9: SW1A, Connector_Wire:SolderWire-0.25sqmm_1x03_P4.2mm_D0.65mm_OD1.7mm, symbol Connector_Generic:Conn_01x03
- removed U3, U4: VTL5C, OptoDevice:PerkinElmer_VTL5C, symbol Isolator:VTL5C
- added J13: 1A1, Connector_Wire:SolderWire-0.25sqmm_1x01_D0.65mm_OD1.7mm, symbol Connector_Generic:Conn_01x01
- added J2: 1A3, Connector_Wire:SolderWire-0.25sqmm_1x01_D0.65mm_OD1.7mm, symbol Connector_Generic:Conn_01x01
- added J20: 1B3, Connector_Wire:SolderWire-0.25sqmm_1x01_D0.65mm_OD1.7mm, symbol Connector_Generic:Conn_01x01
- added J21: 1B2, Connector_Wire:SolderWire-0.25sqmm_1x01_D0.65mm_OD1.7mm, symbol Connector_Generic:Conn_01x01
- added J22: 1B1, Connector_Wire:SolderWire-0.25sqmm_1x01_D0.65mm_OD1.7mm, symbol Connector_Generic:Conn_01x01
- added J23: 1C1, Connector_Wire:SolderWire-0.25sqmm_1x01_D0.65mm_OD1.7mm, symbol Connector_Generic:Conn_01x01
- added J24: 1C2, Connector_Wire:SolderWire-0.25sqmm_1x01_D0.65mm_OD1.7mm, symbol Connector_Generic:Conn_01x01
- added J25: 1C3, Connector_Wire:SolderWire-0.25sqmm_1x01_D0.65mm_OD1.7mm, symbol Connector_Generic:Conn_01x01
- added J9: 1A2, Connector_Wire:SolderWire-0.25sqmm_1x01_D0.65mm_OD1.7mm, symbol Connector_Generic:Conn_01x01
- added V1D1, V2D1: D_Photo, MyLibrary:LED_D5.0mm, symbol MyGlobalLibrary:D_Photo
- added V1R1, V2R1: D_LDR, MyLibrary:R_LDR_5.2x5.2mm_P3.5mm_Horizontal, symbol MyGlobalLibrary:D_LDR
- C2: footprint Capacitor_THT:CP_Radial_D5.0mm_P2.00mm -> MyLibrary:CP_Radial_D5.0mm_PWideForPower
- R22: value 1M8 -> 330r
- SW1: footprint Switches:SWITCH_SPDT_PTH_11.6X4.0MM -> MyLibrary:SWITCH_SPDT_PTH_12.9X6.9MM
Connections:
- net GND: now also RV2.3, J2.1 (Pin_1), J24.1 (Pin_1); no longer RV2.1
- net Mode2: now also RV1.3, V2R1.1; no longer RV1.1
- net Mode3: now also V1R1.1
- net ModeA: now also RV3.1; no longer RV3.3
- net Range8: now also V2R1.2
- net UD6: now also V1D1.1 (K), V2D1.1 (K)
- net UDB: now also RV6.1; no longer RV6.3
- net at C14.1, C16.2, D2.2 (A)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: now also RV3.3; no longer RV3.1
- net at R1.1: now also RV1.1; no longer RV1.3
- net at C14.2, J5.1 (Pin_1), J6.1 (Pin_1): now also RV2.1; no longer RV2.3
- net at R14.1: now also J22.1 (Pin_1)
- net at J10.1 (Pin_1): now also J13.1 (Pin_1), J20.1 (Pin_1)
- net at C15.1: now also J9.1 (Pin_1)
- net at J14.1 (Pin_1): now also J21.1 (Pin_1)
- net at R17.2: now also RV4.3; no longer RV4.1
- net at C20.1, R18.1, RV4.2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: now also RV4.1; no longer RV4.3
- net at R18.2: now also RV5.3; no longer RV5.1
- net at J15.1 (Pin_1), RV5.2: now also RV5.1; no longer RV5.3
- net at J18.1 (Pin_1), R22.2, RV6.2: now also RV6.3; no longer RV6.1
- net at D7.1 (K): now also J23.1 (Pin_1)
- net Vact1-2: no longer names the net of R19.2
- net Vact1-2: now also V1D1.2 (A)
- net Vact1-4: no longer names the net of C6.2, C7.2, C8.2, C9.2, R7.1, U1.2 (-)
- net Vact1-4: now also V1R1.2
- net Vact2-2: no longer names the net of R20.2
- net Vact2-2: now also V2D1.2 (A)
Other:
- note removed: "Vactrols"
- moved on the sheet: J14
